File: Joystick.kicad_pcb (KiCad board)
At the start: 2 copper layers, 157.7 x 102 mm, 10 parts, among them J1 Conn_01x04_Pin, J2 Conn_01x04_Pin, J3 Conn_01x02_Socket, J4 Conn_01x02_Socket, U1 YAAJ_BluePill_Part_Like, U2 NRF24L01_, U3 hw-045

Commit message: production ready
Parts:
- removed J1, J2: Conn_01x04_Pin, Connector_PinHeader_2.54mm:PinHeader_1x04_P2.54mm_Horizontal
- added J5: Conn_01x05_Pin, Connector_PinHeader_2.54mm:PinHeader_1x05_P2.54mm_Horizontal, F.Cu at (124.9, 93.4)
- added J6: Conn_01x05_Pin, Connector_PinHeader_2.54mm:PinHeader_1x05_P2.54mm_Horizontal, F.Cu at (225.9, 94.0)
Connections:
- U1 pad 24: unconnected-(U1-PC15-Pad24) -> /S1
- U1 pad 25: unconnected-(U1-PA0-Pad25) -> /KY
- U1 pad 28: unconnected-(U1-PA3-Pad28) -> /KX
- U1 pad 29: unconnected-(U1-PA4-Pad29) -> /S2
Routing:
- net /S1: track 0.00 -> 124.4 mm
- net /KY: track 0.00 -> 118.0 mm
- net /KX: track 0.00 -> 110.5 mm, vias 0 -> 2
- net /S2: track 0.00 -> 100.2 mm
- net /VIN: track 228.1 -> 212.3 mm
- net /POW: track 72.6 -> 58.2 mm
- net /VX: track 126.6 -> 112.9 mm
- net /VY: track 113.4 -> 103.9 mm
- net Net-(U1-PB10): track 147.6 -> 143.3 mm
- net Net-(U1-PA7): track 125.9 -> 127.0 mm
- net /SCL: track 42.7 -> 43.9 mm
- net /SDL: track 36.4 -> 35.6 mm
