File: Joystick.kicad_sch (KiCad schematic)
At the start: 10 parts, among them J1 Conn_01x04_Pin, J2 Conn_01x04_Pin, J3 Conn_01x02_Socket, J4 Conn_01x02_Socket, U1 YAAJ_BluePill_Part_Like, U2 NRF24L01_, U3 hw-045

Commit message: production ready
Parts:
- removed J1, J2: Conn_01x04_Pin, Connector_PinHeader_2.54mm:PinHeader_1x04_P2.54mm_Horizontal, symbol Connector:Conn_01x04_Pin
- added J5, J6: Conn_01x05_Pin, Connector_PinHeader_2.54mm:PinHeader_1x05_P2.54mm_Horizontal, symbol Connector:Conn_01x05_Pin
Connections:
- net GND: now also J5.1 (Pin_1), J6.1 (Pin_1)
- net VIN: now also J5.2 (Pin_2), J6.2 (Pin_2)
- net VX: now also J6.3 (Pin_3)
- net VY: now also J5.4 (Pin_4)
- net S1: now reaches U1.24 (PC15)
- net S1: now also J6.5 (Pin_5)
- net KY: now reaches U1.25 (PA0)
- net KY: now also J6.4 (Pin_4)
- net KX: now reaches U1.28 (PA3)
- net KX: now also J5.3 (Pin_3)
- net S2: now reaches U1.29 (PA4)
- net S2: now also J5.5 (Pin_5)
- no-connect marks 31 -> 25
